Commit message: Improved collision box for robot

File: src/igus_rebel_ros2/igus_rebel_description/urdf/igus_rebel2.urdf (robot description, URDF)
Before this commit: robot igus_rebel, 18 links, 17 joints
Links:
- link igus_7th_axis: geometry collision box size=1.51 0.42 0.23; visual mesh filename=file://$(find igus_rebel_description)/meshes/robolink_rebel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
