Commit message: Pick and place works with environment

File: install/igus_rebel_description/share/igus_rebel_description/urdf/igus_rebel2.urdf (robot description, URDF)
Before this commit: robot igus_rebel, 15 links, 14 joints
Links:
- link base_tile: geometry collision box size=0.25 0.3 0.025; visual box size=0.25 0.3 0.025
- link igus_7th_axis: geometry collision box size=1.51 0.38 0.23; visual mesh filename=file://$(find igus_rebel_description)/meshes/robolink_rebel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

File: src/igus_rebel_ros2/igus_rebel_description/urdf/igus_rebel2.urdf (robot description, URDF)
Before this commit: robot igus_rebel, 15 links, 14 joints
Links:
- link igus_7th_axis: geometry collision box size=1.51 0.38 0.23; visual mesh filename=file://$(find igus_rebel_description)/meshes/robolink_rebel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

Commit message: Added fixed female part to arm

File: install/igus_rebel_description/share/igus_rebel_description/urdf/igus_rebel2.urdf (robot description, URDF)
Before this commit: robot igus_rebel, 15 links, 14 joints
Links:
- link gripper_link: geometry collision mesh filename=file://$(find igus_rebel_description)/meshes/robolink_rebel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 scale=0.001 0.001 0.001; visual mesh filename=file://$(find igus_rebel_description)/meshes/robolink_rebel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 scale=0.001 0.001 0.001
Joints:
- joint gripper_fixed_joint: origin xyz=0 0 0.053 rpy=0 0 0 -> xyz=0 0 0.053 rpy=-1.57079632679 0 0

Commit message: Pick and place for cup holder and cup

File: install/igus_rebel_description/share/igus_rebel_description/urdf/igus_rebel2.urdf (robot description, URDF)
Before this commit: robot igus_rebel, 15 links, 14 joints
Links:
- link gripper_link: geometry collision mesh filename=file://$(find igus_rebel_description)/meshes/robolink_rebel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; visual mesh filename=file://$(find igus_rebel_description)/meshes/robolink_rebel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 scale=0.001 0.001 0.001
