Commit message: Pick and place is done higher up

File: install/igus_rebel_description/share/igus_rebel_description/urdf/igus_rebel2.control.xacro (robot description, xacro)
@@ -37,6 +37,4 @@
             <xacro:joint_control joint="joint5" />
             <xacro:joint_control joint="joint6" />
-            <xacro:joint_control joint="left_finger_joint" />   <!-- ADD THIS -->
-            <xacro:joint_control joint="right_finger_joint" />
         </ros2_control>
         <xacro:if value="${hardware_protocol == 'gazebo'}">

File: install/igus_rebel_description/share/igus_rebel_description/urdf/igus_rebel2.urdf (robot description, URDF)
Before this commit: robot igus_rebel, 18 links, 17 joints
Links:
- removed link gripper_mount
- removed link left_finger
- removed link right_finger
- removed link tcp
- added link gripper_link; collision mesh filename=file://$(find igus_rebel_description)/meshes/robolink_rebel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; visual mesh filename=file://$(find igus_rebel_description)/meshes/robolink_rebel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
- link base_tile: geometry visual box size=0.25 0.3 0.025
- link igus_7th_axis: geometry visual mesh filename=file://$(find igus_rebel_description)/meshes/robolink_rebel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
Joints:
- removed joint gripper_mount_joint
- removed joint left_finger_joint
- removed joint right_finger_joint
- removed joint tcp_joint
- added joint gripper_fixed_joint: type fixed, parent link6, child gripper_link, origin xyz=0 0 0.053 rpy=0 0 0

File: src/igus_rebel_ros2/igus_rebel_description/urdf/igus_rebel2.urdf (robot description, URDF)
Before this commit: robot igus_rebel, 15 links, 14 joints
Links:
- link igus_7th_axis: geometry collision box size=1.51 1.02 0.23; visual mesh filename=file://$(find igus_rebel_description)/meshes/robolink_rebel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

Commit message: Removed rail

File: install/igus_rebel_description/share/igus_rebel_description/urdf/igus_rebel2.control.xacro (robot description, xacro)
@@ -27,8 +27,7 @@
                 </xacro:if>
                 <parameters>
-                    <param name="update_rate">100</param> <!-- Change to desired rate (Hz) -->
+                    <param name="update_rate">100</param>
                 </parameters>
             </hardware>
-            <xacro:joint_control joint="rail_slider" />
             <xacro:joint_control joint="joint1" />
             <xacro:joint_control joint="joint2" />

File: install/igus_rebel_description/share/igus_rebel_description/urdf/igus_rebel2.urdf (robot description, URDF)
Before this commit: robot igus_rebel, 15 links, 14 joints
Links:
- removed link base_tile
- removed link igus_7th_axis
Joints:
- removed joint rail_slider
- removed joint robot_on_tile

File: install/igus_rebel_description/share/igus_rebel_description/urdf1/igus_rebel.control.xacro (robot description, xacro)
@@ -15,5 +15,4 @@
             </transmission>
         </xacro:macro>
-        <xacro:arm_control transmission="${arm_id}_tran_0" joint="rail_slider" motor="${arm_id}_motor_0"/>
         <xacro:arm_control transmission="${arm_id}_tran_1" joint="joint1" motor="${arm_id}_motor_1"/>
         <xacro:arm_control transmission="${arm_id}_tran_2" joint="joint2" motor="${arm_id}_motor_2"/>

File: install/igus_rebel_description/share/igus_rebel_description/urdf1/igus_rebel_robot.urdf.xacro (robot description, xacro)
@@ -3,5 +3,4 @@
        name="igus_rebel" >
   <xacro:arg name="hardware_protocol" default="rebel"/>
-  <!-- igus_rebel -->
   <xacro:include filename="$(find igus_rebel_description)/urdf/igus_rebel2.urdf" />
   <xacro:include filename="$(find igus_rebel_description)/urdf/igus_rebel2.control.xacro"/>
@@ -10,6 +9,5 @@
   <joint name="world_joint" type="fixed">
     <parent link="world" />
-    <child link = "igus_7th_axis" />
-    <!-- <child link = "base_link" /> -->
+    <child link="base_link" />
     <origin xyz="0.0 0.0 0.0" rpy="0.0 0.0 0.0" />
   </joint>
