Commit message: Done four tasks

File: install/igus_rebel_description/share/igus_rebel_description/urdf1/igus_rebel_robot.urdf.xacro (robot description, xacro)
@@ -10,5 +10,5 @@
     <parent link="world" />
     <child link="base_link" />
-    <origin xyz="0.0 0.0 0.0" rpy="0.0 0.0 0.0" />
+    <origin xyz="0.0 0.0 0.0" rpy="0.0 0.0 -1.5707963268" />
   </joint>
 </robot>
